Commit message: Maly lazik w URDF-ach, zmiany rozmiarow i polozenie

File: src/trailblazer_description/urdf/depth_camera.xacro (robot description, xacro)
@@ -4,5 +4,5 @@
         <parent link="chassis"/>
         <child link="camera_link"/>
-        <origin xyz="0.001 0.146 0.4465" rpy="0 -1.5708 0"/>
+        <origin xyz="0.001 0.126 0.1275" rpy="0 -1.5708 0"/>
     </joint>
     <link name="camera_link">

File: src/trailblazer_description/urdf/gazebo_control.xacro (robot description, xacro)
@@ -6,6 +6,6 @@
             <left_joint>FL_wheel_joint</left_joint>
             <right_joint>FR_wheel_joint</right_joint>
-            <wheel_separation>1.17</wheel_separation>
-            <wheel_diameter>0.26</wheel_diameter>
+            <wheel_separation>0.225</wheel_separation>
+            <wheel_diameter>0.065</wheel_diameter>
             <!-- Limit -->
             <max_wheel_torque>200</max_wheel_torque>
@@ -25,6 +25,6 @@
             <left_joint>BL_wheel_joint</left_joint>
             <right_joint>BR_wheel_joint</right_joint>
-            <wheel_separation>1.17</wheel_separation>
-            <wheel_diameter>0.26</wheel_diameter>
+            <wheel_separation>0.225</wheel_separation>
+            <wheel_diameter>0.065</wheel_diameter>
             <!-- Limit -->
             <max_wheel_torque>200</max_wheel_torque>

File: src/trailblazer_description/urdf/imu.xacro (robot description, xacro)
@@ -4,5 +4,5 @@
         <parent link="chassis"/>
         <child link="imu_link"/>
-        <origin xyz="0.001 0.146 0.4465" rpy="0 -1.5708 0"/>
+        <origin xyz="0.001 0.126 0.1275" rpy="0 -1.5708 0"/>
     </joint>
     <link name="imu_link">

File: src/trailblazer_description/urdf/rover.urdf.xacro (robot description, xacro)
@@ -56,5 +56,5 @@
   <link
     name="chassis">
-    <inertial>
+    <!-- <inertial>
       <origin
         xyz="0.00322150223165306 -0.0317835441688463 0.0392262662545424"
@@ -69,32 +69,37 @@
         iyz="1.36293755133581E-06"
         izz="0.0668521247692141" />
-    </inertial>
-    <visual>
-      <origin
-        xyz="0 0 0"
-        rpy="0 0 0" />
-      <geometry>
-        <mesh
-          filename="package://trailblazer_description/meshes/base_link.STL" />
-      </geometry>
-      <material
-        name="">
-        <color
-          rgba="0.752941176470588 0.752941176470588 0.752941176470588 1" />
-      </material>
-    </visual>
-    <collision>
-      <origin
-        xyz="0 0 0"
-        rpy="0 0 0" />
-      <geometry>
-        <mesh
-          filename="package://trailblazer_description/meshes/base_link.STL" />
-      </geometry>
-    </collision>
+    </inertial> -->
+    <visual>
+      <origin
+        xyz="0 0.09 0"
+        rpy="0 0 0" />
+      <geometry>
+        <!-- <mesh
+          filename="package://trailblazer_description/meshes/base_link.STL" /> -->
+        <box size="0.20 0.115 0.225"/>
+      </geometry>
+      <material
+        name="">
+        <color
+          rgba="0.752941176470588 0.752941176470588 0.752941176470588 1" />
+      </material>
+    </visual>
+    <collision>
+      <origin
+        xyz="0 0.09 0"
+        rpy="0 0 0" />
+      <geometry>
+        <!-- <mesh
+          filename="package://trailblazer_description/meshes/base_link.STL" /> -->
+        <box size="0.20 0.115 0.225"/>
+      </geometry>
+    </collision>
+    <xacro:inertial_box mass="0.5" x="0.20" y="0.115" z="0.225">
+      <origin xyz="0 0.09 0"/>
+    </xacro:inertial_box>
   </link>
   <link
     name="FL_wheel">
-    <inertial>
+    <!-- <inertial>
       <origin
         xyz="-0.0657932903439138 0.00142869200681425 9.9374601122415E-06"
@@ -109,28 +114,33 @@
         iyz="7.8978424094368E-07"
         izz="0.0076927565336923" />
-    </inertial>
-    <visual>
-      <origin
-        xyz="0 0 0"
-        rpy="0 0 0" />
-      <geometry>
-        <mesh
-          filename="package://trailblazer_description/meshes/FL_wheel.STL" />
-      </geometry>
-      <material
-        name="">
-        <color
-          rgba="0.752941176470588 0.752941176470588 0.752941176470588 1" />
-      </material>
-    </visual>
-    <collision>
-      <origin
-        xyz="0 0 0"
-        rpy="0 0 0" />
-      <geometry>
-        <mesh
-          filename="package://trailblazer_description/meshes/FL_wheel.STL" />
-      </geometry>
-    </collision>
+    </inertial> -->
+    <visual>
+      <origin
+        xyz="0 0 0"
+        rpy="0 -${pi/2} 0" />
+      <geometry>
+        <!-- <mesh
+          filename="package://trailblazer_description/meshes/FL_wheel.STL" /> -->
+        <cylinder radius="0.035" length="0.025"/>
+      </geometry>
+      <material
+        name="">
+        <color
+          rgba="0.752941176470588 0.752941176470588 0.752941176470588 1" />
+      </material>
+    </visual>
+    <collision>
+      <origin
+        xyz="0 0 0"
+        rpy="0 -${pi/2} 0" />
+      <geometry>
+        <!-- <mesh
+          filename="package://trailblazer_description/meshes/FL_wheel.STL" /> -->
+        <cylinder radius="0.035" length="0.025"/>
+      </geometry>
+    </collision>
+    <xacro:inertial_cylinder mass="0.01" radius="0.035" length="0.025">
+      <origin xyz="0 0 0"/>
+    </xacro:inertial_cylinder>
   </link>
   <joint
@@ -138,5 +148,5 @@
     type="continuous">
     <origin
-      xyz="0.578691303668632 -0.237965989839832 0.501750000756599"
+      xyz="0.1125 0.035 0.1025"
       rpy="0 0 0" />
     <parent
@@ -149,5 +159,5 @@
   <link
     name="BL_wheel">
-    <inertial>
+    <!-- <inertial>
       <origin
         xyz="-0.0657953215031118 0.00133190879616998 -1.102290957955E-06"
@@ -162,28 +172,33 @@
         iyz="6.94182413139629E-08"
         izz="0.00769259835014326" />
-    </inertial>
-    <visual>
-      <origin
-        xyz="0 0 0"
-        rpy="0 0 0" />
-      <geometry>
-        <mesh
-          filename="package://trailblazer_description/meshes/BL_wheel.STL" />
-      </geometry>
-      <material
-        name="">
-        <color
-          rgba="0.752941176470588 0.752941176470588 0.752941176470588 1" />
-      </material>
-    </visual>
-    <collision>
-      <origin
-        xyz="0 0 0"
-        rpy="0 0 0" />
-      <geometry>
-        <mesh
-          filename="package://trailblazer_description/meshes/BL_wheel.STL" />
-      </geometry>
-    </collision>
+    </inertial> -->
+    <visual>
+      <origin
+        xyz="0 0 0"
+        rpy="0 -${pi/2} 0" />
+      <geometry>
+        <!-- <mesh
+          filename="package://trailblazer_description/meshes/BL_wheel.STL" /> -->
+        <cylinder radius="0.035" length="0.025"/>
+      </geometry>
+      <material
+        name="">
+        <color
+          rgba="0.752941176470588 0.752941176470588 0.752941176470588 1" />
+      </material>
+    </visual>
+    <collision>
+      <origin
+        xyz="0 0 0"
+        rpy="0 -${pi/2} 0" />
+      <geometry>
+        <!-- <mesh
+          filename="package://trailblazer_description/meshes/BL_wheel.STL" /> -->
+        <cylinder radius="0.035" length="0.025"/>
+      </geometry>
+    </collision>
+    <xacro:inertial_cylinder mass="0.01" radius="0.035" length="0.025">
+      <origin xyz="0 0 0"/>
+    </xacro:inertial_cylinder>
   </link>
   <joint
@@ -191,5 +206,5 @@
     type="continuous">
     <origin
-      xyz="0.578691303668647 -0.237965989839099 -0.401750000000183"
+      xyz="0.1125 0.035 -0.1025"
       rpy="0 0 0" />
     <parent
@@ -202,5 +217,5 @@
   <link
     name="FR_wheel">
-    <inertial>
+    <!-- <inertial>
       <origin
         xyz="0.0657913230041458 0.0013308416445233 8.05670440151562E-06"
@@ -215,28 +230,33 @@
         iyz="-6.97714576728623E-07"
         izz="0.00769272793356072" />
-    </inertial>
-    <visual>
-      <origin
-        xyz="0 0 0"
-        rpy="0 0 0" />
-      <geometry>
-        <mesh
-          filename="package://trailblazer_description/meshes/FR_wheel.STL" />
-      </geometry>
-      <material
-        name="">
-        <color
-          rgba="0.752941176470588 0.752941176470588 0.752941176470588 1" />
-      </material>
-    </visual>
-    <collision>
-      <origin
-        xyz="0 0 0"
-        rpy="0 0 0" />
-      <geometry>
-        <mesh
-          filename="package://trailblazer_description/meshes/FR_wheel.STL" />
-      </geometry>
-    </collision>
+    </inertial> -->
+    <visual>
+      <origin
+        xyz="0 0 0"
+        rpy="0 -${pi/2} 0" />
+      <geometry>
+        <!-- <mesh
+          filename="package://trailblazer_description/meshes/FR_wheel.STL" /> -->
+        <cylinder radius="0.035" length="0.025"/>
+      </geometry>
+      <material
+        name="">
+        <color
+          rgba="0.752941176470588 0.752941176470588 0.752941176470588 1" />
+      </material>
+    </visual>
+    <collision>
+      <origin
+        xyz="0 0 0"
+        rpy="0 -${pi/2} 0" />
+      <geometry>
+        <!-- <mesh
+          filename="package://trailblazer_description/meshes/FR_wheel.STL" /> -->
+        <cylinder radius="0.035" length="0.025"/>
+      </geometry>
+    </collision>
+    <xacro:inertial_cylinder mass="0.01" radius="0.035" length="0.025">
+      <origin xyz="0 0 0"/>
+    </xacro:inertial_cylinder>
   </link>
   <joint
@@ -244,5 +264,5 @@
     type="continuous">
     <origin
-      xyz="-0.578691303668549 -0.237965989839575 0.50175"
+      xyz="-0.1125 0.035 0.1025"
       rpy="0 0 0" />
     <parent
@@ -255,5 +275,5 @@
   <link
     name="BR_wheel">
-    <inertial>
+    <!-- <inertial>
       <origin
         xyz="0.0657913365617738 0.00133019561822817 -1.39445307800745E-07"
@@ -268,28 +288,33 @@
         iyz="-5.04460531278865E-08"
         izz="0.00769260505729232" />
-    </inertial>
-    <visual>
-      <origin
-        xyz="0 0 0"
-        rpy="0 0 0" />
-      <geometry>
-        <mesh
-          filename="package://trailblazer_description/meshes/BR_wheel.STL" />
-      </geometry>
-      <material
-        name="">
-        <color
-          rgba="0.752941176470588 0.752941176470588 0.752941176470588 1" />
-      </material>
-    </visual>
-    <collision>
-      <origin
-        xyz="0 0 0"
-        rpy="0 0 0" />
-      <geometry>
-        <mesh
-          filename="package://trailblazer_description/meshes/BR_wheel.STL" />
-      </geometry>
-    </collision>
+    </inertial> -->
+    <visual>
+      <origin
+        xyz="0 0 0"
+        rpy="0 -${pi/2} 0" />
+      <geometry>
+        <!-- <mesh
+          filename="package://trailblazer_description/meshes/BR_wheel.STL" /> -->
+        <cylinder radius="0.035" length="0.025"/>
+      </geometry>
+      <material
+        name="">
+        <color
+          rgba="0.752941176470588 0.752941176470588 0.752941176470588 1" />
+      </material>
+    </visual>
+    <collision>
+      <origin
+        xyz="0 0 0"
+        rpy="0 -${pi/2} 0" />
+      <geometry>
+        <!-- <mesh
+          filename="package://trailblazer_description/meshes/BR_wheel.STL" /> -->
+        <cylinder radius="0.035" length="0.025"/>
+      </geometry>
+    </collision>
+    <xacro:inertial_cylinder mass="0.01" radius="0.035" length="0.025">
+      <origin xyz="0 0 0"/>
+    </xacro:inertial_cylinder>
   </link>
   <joint
@@ -297,5 +322,5 @@
     type="continuous">
     <origin
-      xyz="-0.578691303668548 -0.237965989839575 -0.401750000756777"
+      xyz="-0.1125 0.035 -0.1025"
       rpy="0 0 0" />
     <parent
